File: Schematic/Schematic.kicad_sch (KiCad schematic)
At the start: 2 parts, among them J1 Conn_02x17_Top_Bottom, J2 Conn_01x08_Pin

Commit message: updated schematic
Parts:
- added BT1: 6V Battery, symbol Device:Battery
- added C1: 0.33uF, symbol Device:C
- added C2, C3, C4: 0.1uF, symbol Device:C
- added M1: Motor_Servo, symbol Motor:Motor_Servo
- added R1, R2: 10k, symbol Device:R
- added SW1: SW_DPDT_x2, symbol Switch:SW_DPDT_x2
- added SW2, SW3: SW_Push, symbol Switch:SW_Push
- added U1: L7805, symbol Regulator_Linear:L7805
Connections:
- net 0: now also C4.1, R2.1, SW3.1
- net 21: now also M1.1 (PWM)
- net 4: now also C3.1, R1.1, SW2.1
- net 5V: now also C2.1, C3.2, C4.2, SW1.1 (A), SW1.2 (B), SW2.2, SW3.2, U1.3 (OUT)
- net GND: now also BT1.2 (-), C1.2, C2.2, M1.3 (-), R1.2, R2.2, U1.2 (GND)
- new net 6V: BT1.1 (+), C1.1, M1.2 (+), U1.1 (IN)
Other:
- note added: "5 - SDA 18 - SCK 23 - MOSI 19 - MISO 10 - RST"
- note added: "Switch to disconnect power if rewriting to ESP32"
- moved on the sheet: J1, J2
